File: Hardware/Brewpilessboard.sch (KiCad schematic (older format))
At the start: 6 parts, among them U1 ESP32_DevKit_V1_DOIT

Commit message: Further changes to board layout
Parts:
- added A1: I2Cconn, Connector_PinSocket_2.54mm:PinSocket_1x04_P2.54mm_Horizontal, symbol brewpilessboardsymbols:I2Cconn
- added F1: Fuse, Fuse:Fuse_1206_3216Metric_Pad1.42x1.75mm_HandSolder, symbol Device:Fuse
- added J1, J2: Conn_01x01_Female, Connector_PinHeader_2.54mm:PinHeader_1x01_P2.54mm_Vertical, symbol Connector:Conn_01x01_Female
- K1: renamed from K?; footprint (none) -> Libraries:2channelrelayboard3.9x5.1cm
- PS1: renamed from PS?; footprint CONV_HLK-5M05 -> Libraries:CONV_HLK-5M05
- R1: renamed from R?; footprint (none) -> Resistor_THT:R_Axial_DIN0204_L3.6mm_D1.6mm_P7.62mm_Horizontal
- U2, U3: renamed from U?; footprint Package_TO_SOT_THT:TO-92_Inline -> Connector_PinSocket_2.54mm:PinSocket_1x03_P2.54mm_Vertical
Connections:
- net +5V: now also R1.1, U2.3 (VDD), U3.3 (VDD); no longer U1.15 (VIN)
- net GND: now also A1.2 (GND)
- net NEUT: now also J2.1 (Pin_1)
- net VAC: now also F1.2
- net SDA: now reaches U1.26 (IO21)
- net SDA: now also A1.3 (SDA)
- net SCL: now reaches U1.29 (IO22)
- net SCL: now also A1.4 (SCL)
- net OneWire: now reaches R1.2, U1.30 (IO23), U2.2 (DQ), U3.2 (DQ)
- new net: F1.1, J1.1 (Pin_1)
- new net +3V3: A1.1 (3.3VDC)
- now unconnected: U1.16 (3V3)
- no-connect marks 0 -> 21
Other:
- note added: "240VAC"
- note added: "240VAC/5VDC buck converter"
- note added: "DS18B20 Onewire Temp Sensors"
- note added: "Relay"
- note added: "Screen connector"

Commit message: Further changes
Parts:
- removed J1, J2: Conn_01x01_Female, Connector_PinHeader_2.54mm:PinHeader_1x01_P2.54mm_Vertical, symbol Connector:Conn_01x01_Female
- added C1, C2, C3, C4: 0.1u, Capacitor_SMD:C_1206_3216Metric_Pad1.42x1.75mm_HandSolder, symbol Device:C_Small
- added J4: Conn_01x02_Male, Connector_JST:JST_XH_B2B-XH-AM_1x02_P2.50mm_Vertical, symbol Connector:Conn_01x02_Male
- R1: footprint Resistor_THT:R_Axial_DIN0204_L3.6mm_D1.6mm_P7.62mm_Horizontal -> Resistor_SMD:R_1206_3216Metric_Pad1.42x1.75mm_HandSolder
Connections:
- net labels added: +3V3, IN1, IN2
- net labels removed: +3.3V
- wire segments 19 -> 23
Other:
- note added: "Power in and rectification/transformer"
- note removed: "240VAC"
- note removed: "240VAC/5VDC buck converter"
- moved on the sheet: A1, F1, K1, PS1, R1, U1, U2, U3
